File: TTK4155-Embedded-PCB.kicad_pcb (KiCad board)
At the start: 2 copper layers, 42 parts, among them J1 AVR-JTAG-10, J2 DB9_Female, J3 Conn_01x10_Male, J4 Conn_01x04_Male, J5 Screw_Terminal_01x02, J6 Screw_Terminal_01x02, SW1 SW_Push, U1 L7805, U2 ATmega162-16PU, U3 IDT7164S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

Commit message: Finished first revision of board
Parts:
- added J7: Conn_01x04_Male, Connector_PinHeader_2.54mm:PinHeader_1x04_P2.54mm_Vertical, F.Cu at (74.3, 49.8)
- added J8: BannanaJack, TTK4155-Embedded-PCB:Banana_Jack_2Pin_15mm_spacing, F.Cu at (135.9, 105.0)
- moved J1 12.2 mm to (98.6, 127.9), turned to 90 degrees
- moved J6 10.2 mm to (122.9, 127.1)
- moved J2 7.62 mm to (82.4, 119.8)
- moved R1 2.50 mm to (77.0, 37.0), turned to 180 degrees
- moved C14 2.44 mm to (103.3, 69.0)
- moved R2 1.89 mm to (82.3, 34.7)
- moved C3 1.89 mm to (82.0, 38.2)
- moved J4 0.25 mm to (112.9, 88.0)
Connections:
- J6 pad 1: Net-(J6-Pad1) -> +12V
Routing:
- net +5V: track 0.00 -> 299.8 mm, vias 0 -> 8
- net /~RESET: track 0.00 -> 107.4 mm
- net /TDI: track 0.00 -> 79.1 mm, vias 0 -> 1
- net /~OE: track 0.00 -> 78.1 mm, vias 0 -> 1
- net /TDO: track 0.00 -> 67.3 mm, vias 0 -> 2
- net /TMS: track 0.00 -> 64.7 mm, vias 0 -> 1
- net /INT0: track 0.00 -> 64.2 mm, vias 0 -> 1
- net /CS_RAM: track 0.00 -> 60.7 mm, vias 0 -> 2
- net +12V: track 0.00 -> 60.0 mm
- net /TCK: track 0.00 -> 53.8 mm, vias 0 -> 1
- net /TXD0: track 0.00 -> 39.6 mm
- net /RXD0: track 0.00 -> 38.1 mm
- net /~RESETCAN: track 0.00 -> 36.1 mm
- net /RXCAN: track 0.00 -> 35.6 mm
- net /OLED_DATA: track 0.00 -> 34.2 mm
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- added copper zone on B.Cu, net GND
- added copper zone on F.Cu, net GND
Other:
- board outline added: 100 x 100 mm
- board text added: "+"
- board text added: "Buttons"
- board text added: "GND"
- board text added: "OLED Memory and controller"
- board text added: "RESET"
- board text added: "Sliders and Joystick"
- board text added: "TTK4155 - Node 1 Ole Sivert Aarhaug Audun Asdal Einar Marstrander Omang"

Commit message: Fixed missing pullup
Parts:
- added R7: 10K, Resistor_SMD:R_0805_2012Metric_Pad1.15x1.40mm_HandSolder, F.Cu at (77.0, 39.2)
Routing:
- net +5V: track 299.8 -> 306.4 mm, vias 8 -> 9
- net Net-(J7-Pad4): track 3.43 -> 7.03 mm
Changed lines of the file:
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@@
     (thickness 1.6)
     (drawings 17)
-    (tracks 543)
+    (tracks 549)
     (zones 0)
-    (modules 44)
+    (modules 45)
     (nets 106)
   )
@@
     (solder_mask_min_width 0.25)
     (aux_axis_origin 0 0)
-    (visible_elements FFFFFF7F)
+    (visible_elements 7FFFFFFF)
     (pcbplotparams
-      (layerselection 0x010fc_ffffffff)
+      (layerselection 0x010f0_ffffffff)
       (usegerberextensions false)
       (usegerberattributes false)
       (usegerberadvancedattributes false)
       (creategerberjobfile false)
-      (excludeedgelayer true)
+      (excludeedgelayer false)
       (linewidth 0.100000)
       (plotframeref false)
@@
       (outputformat 1)
       (mirror false)
-      (drillshape 1)
+      (drillshape 0)
       (scaleselection 1)
-      (outputdirectory ""))
+      (outputdirectory "gerber/"))
   )
   (net 0 "")
@@
     (add_net "Net-(U8-Pad8)")
   )
+  (module Resistor_SMD:R_0805_2012Metric_Pad1.15x1.40mm_HandSolder (layer F.Cu)
+    (at 76.962 39.243 180)
+    (descr "Resistor SMD 0805 (2012 Metric), square (rectangular) end terminal, IPC_7351 nominal with elongated pad for handsoldering. (Body size source: https://docs.google.com/spreadsheets/d/1BsfQQcO9C6DZCsRaXUlFlo91Tg2WpOkGARC1WS5S8t0/edit?usp=sharing), generated with kicad-footprint-generator")
+    (tags "resistor handsolder")
+    (attr smd)
+    (fp_text reference R7 (at -2.54 0.254 270) (layer F.SilkS)
+      (effects (font (size 1 1) (thickness 0.15)))
+    )
+    (fp_text value 10K (at 3.175 -0.254) (layer F.SilkS)
+      (effects (font (size 1 1) (thickness 0.15)))
+    )
+    (fp_text user %R (at 0 0) (layer F.Fab)
+      (effects (font (size 0.5 0.5) (thickness 0.08)))
+    )
+    (fp_line (start 1.85 0.95) (end -1.85 0.95) (layer F.CrtYd) (width 0.05))
+    (fp_line (start 1.85 -0.95) (end 1.85 0.95) (layer F.CrtYd) (width 0.05))
+    (fp_line (start -1.85 -0.95) (end 1.85 -0.95) (layer F.CrtYd) (width 0.05))
+    (fp_line (start -1.85 0.95) (end -1.85 -0.95) (layer F.CrtYd) (width 0.05))
+    (fp_line (start -0.261252 0.71) (end 0.261252 0.71) (layer F.SilkS) (width 0.12))
+    (fp_line (start -0.261252 -0.71) (end 0.261252 -0.71) (layer F.SilkS) (width 0.12))
+    (fp_line (start 1 0.6) (end -1 0.6) (layer F.Fab) (width 0.1))
+    (fp_line (start 1 -0.6) (end 1 0.6) (layer F.Fab) (width 0.1))
+    (fp_line (start -1 -0.6) (end 1 -0.6) (layer F.Fab) (width 0.1))
+    (fp_line (start -1 0.6) (end -1 -0.6) (layer F.Fab) (width 0.1))
+    (pad 2 smd roundrect (at 1.025 0 180) (size 1.15 1.4) (layers F.Cu F.Paste F.Mask) (roundrect_rratio 0.217391)
+      (net 102 "Net-(J7-Pad4)"))
+    (pad 1 smd roundrect (at -1.025 0 180) (size 1.15 1.4) (layers F.Cu F.Paste F.Mask) (roundrect_rratio 0.217391)
+      (net 2 +5V))
+    (model ${KISYS3DMOD}/Resistor_SMD.3dshapes/R_0805_2012Metric.wrl
+      (at (xyz 0 0 0))
+      (scale (xyz 1 1 1))
+      (rotate (xyz 0 0 0))
+    )
+  )
   (module TTK4155-Embedded-PCB:Banana_Jack_2Pin_15mm_spacing (layer F.Cu)
     (at 135.89 105.029 270)
@@
     (tags "resistor handsolder")
     (attr smd)
-    (fp_text reference R1 (at 0 -1.65) (layer F.SilkS)
+    (fp_text reference R1 (at 2.794 0.127) (layer F.SilkS)
       (effects (font (size 1 1) (thickness 0.15)))
     )
@@
   (segment (start 88.011 47.117) (end 88.764 46.364) (width 0.25) (layer B.Cu) (net 2))
   (segment (start 88.011 51.181) (end 88.011 47.117) (width 0.25) (layer B.Cu) (net 2))
+  (segment (start 81.271 34.671) (end 81.271 37.093) (width 0.25) (layer B.Cu) (net 2))
+  (via (at 77.987 39.243) (size 0.8) (drill 0.4) (layers F.Cu B.Cu) (net 2))
+  (segment (start 81.271 37.093) (end 79.121 39.243) (width 0.25) (layer B.Cu) (net 2))
+  (segment (start 79.121 39.243) (end 77.987 39.243) (width 0.25) (layer B.Cu) (net 2))
   (segment (start 81.017 36.975) (end 83.321 34.671) (width 0.25) (layer F.Cu) (net 3))
   (segment (start 81.017 38.227) (end 81.017 36.975) (width 0.25) (layer F.Cu) (net 3))
@@
   (segment (start 109.22 49.784) (end 110.67 49.784) (width 0.25) (layer F.Cu) (net 101))
   (segment (start 77.724 42.164) (end 74.295 42.164) (width 0.25) (layer F.Cu) (net 102))
+  (segment (start 75.937 40.522) (end 74.295 42.164) (width 0.25) (layer F.Cu) (net 102))
+  (segment (start 75.937 39.243) (end 75.937 40.522) (width 0.25) (layer F.Cu) (net 102))
   (segment (start 77.724 44.704) (end 74.295 44.704) (width 0.25) (layer F.Cu) (net 103))
   (segment (start 76.59263 47.244) (end 74.295 47.244) (width 0.25) (layer F.Cu) (net 104))

Commit message: Made som esmall changes and send pcb to production
Parts:
- added R10: 10K, Resistor_SMD:R_0805_2012Metric_Pad1.15x1.40mm_HandSolder, F.Cu at (70.5, 49.3)
- added R8: 10K, Resistor_SMD:R_0805_2012Metric_Pad1.15x1.40mm_HandSolder, F.Cu at (70.5, 44.6)
- added R9: 10K, Resistor_SMD:R_0805_2012Metric_Pad1.15x1.40mm_HandSolder, F.Cu at (70.5, 47.2)
- moved R7 0.13 mm to (77.1, 39.2), turned to 0 degrees
Connections:
- net Net-(J7-Pad1) renamed /PB3
- net Net-(J7-Pad2) renamed /PB2
- net Net-(J7-Pad3) renamed /PB1
- J7 pad 4: Net-(J7-Pad4) -> /PB0
- R7 pad 1: +5V -> /PB0
- R7 pad 2: Net-(J7-Pad4) -> +5V
- U2 pad 1: Net-(J7-Pad4) -> /PB0
Routing:
- net +5V: track 306.4 -> 313.9 mm
- net Net-(J7-Pad4): track 7.03 -> 0.00 mm
- net /PB0: track 0.00 -> 7.03 mm
- net /PB3: track 3.43 -> 6.40 mm, vias 0 -> 1
- net /PB1: track 3.43 -> 6.27 mm, vias 0 -> 1
- net /PB2: track 3.43 -> 6.24 mm, vias 0 -> 1
