File: node2/node2/node2.sch (KiCad schematic (older format))
At the start: 14 parts, among them K1 FINDER-40.52, Q1 MPSA92, U1 MCP602

Commit message: small fixes in node2
Parts:
- D2: value IR204A -> IR LED
- K1: value FINDER-40.52 -> RG2L-5VDC
- Q1: value MPSA92 -> MPSA56
- R2: value R_PHOTO -> IR_PHOTO
Other:
- moved on the sheet: D1, R6
Changed lines of the file:
@@
 P 5150 1900
 F 0 "Q1" H 5341 1854 50  0000 L CNN
-F 1 "MPSA92" H 5341 1945 50  0000 L CNN
+F 1 "MPSA56" H 5341 1945 50  0000 L CNN
 F 2 "Package_TO_SOT_THT:TO-92_Inline" H 5350 1825 50  0001 L CIN
 F 3 "http://www.onsemi.com/pub_link/Collateral/MPSA92-D.PDF" H 5150 1900 50  0001 L CNN
@@
 $EndComp
 $Comp
-L LED:IR204A D2
-U 1 1 5DCFF8D1
-P 7800 5750
-F 0 "D2" H 7750 6040 50  0000 C CNN
-F 1 "IR204A" H 7750 5949 50  0000 C CNN
-F 2 "LED_THT:LED_D3.0mm_IRBlack" H 7800 5925 50  0001 C CNN
-F 3 "http://www.everlight.com/file/ProductFile/IR204-A.pdf" H 7750 5750 50  0001 C CNN
-	1    7800 5750
-	0    -1   -1   0
-$EndComp
-$Comp
 L Device:R_PHOTO R2
 U 1 1 5DD00899
 P 7800 3900
 F 0 "R2" H 7870 3946 50  0000 L CNN
-F 1 "R_PHOTO" H 7870 3855 50  0000 L CNN
+F 1 "IR_PHOTO" H 7870 3855 50  0000 L CNN
 F 2 "" V 7850 3650 50  0001 L CNN
 F 3 "~" H 7800 3850 50  0001 C CNN
@@
 	7200 2500 7750 2500
 Wire Wire Line
-	6350 2100 6750 2100
-Wire Wire Line
-	6750 2100 7200 2100
-Connection ~ 6750 2100
-Connection ~ 6350 2600
-Wire Wire Line
-	6350 2600 7750 2600
-Wire Wire Line
-	6050 2600 6350 2600
-Connection ~ 6350 2100
-Wire Wire Line
-	6350 2200 6350 2100
-Wire Wire Line
-	6050 2100 6350 2100
-Wire Wire Line
 	5450 2500 5200 2500
 $Comp
@@
 P 5750 2500
 F 0 "K1" V 4983 2500 50  0000 C CNN
-F 1 "FINDER-40.52" V 5074 2500 50  0000 C CNN
+F 1 "RG2L-5VDC" V 5074 2500 50  0000 C CNN
 F 2 "Relay_THT:Relay_DPDT_Finder_40.52" H 7100 2470 50  0001 C CNN
 F 3 "http://gfinder.findernet.com/assets/Series/353/S40EN.pdf" H 5550 2500 50  0001 C CNN
@@
 L pspice:DIODE D1
 U 1 1 5DD1E4AA
-P 6350 2400
-F 0 "D1" V 6396 2272 50  0000 R CNN
-F 1 "DIODE" V 6305 2272 50  0000 R CNN
-F 2 "" H 6350 2400 50  0001 C CNN
-F 3 "~" H 6350 2400 50  0001 C CNN
-	1    6350 2400
+P 6600 2400
+F 0 "D1" V 6646 2272 50  0000 R CNN
+F 1 "DIODE" V 6555 2272 50  0000 R CNN
+F 2 "" H 6600 2400 50  0001 C CNN
+F 3 "~" H 6600 2400 50  0001 C CNN
+	1    6600 2400
 	0    1    1    0
 $EndComp
@@
 L power:GND #PWR0108
 U 1 1 5DD150B6
-P 6750 2100
-F 0 "#PWR0108" H 6750 1850 50  0001 C CNN
-F 1 "GND" H 6755 1927 50  0000 C CNN
-F 2 "" H 6750 2100 50  0001 C CNN
-F 3 "" H 6750 2100 50  0001 C CNN
-	1    6750 2100
+P 6900 2100
+F 0 "#PWR0108" H 6900 1850 50  0001 C CNN
+F 1 "GND" H 6905 1927 50  0000 C CNN
+F 2 "" H 6900 2100 50  0001 C CNN
+F 3 "" H 6900 2100 50  0001 C CNN
+	1    6900 2100
 	1    0    0    -1
 $EndComp
@@
 U 2 1 5DCF8177
 P 6000 4050
-F 0 "U1" H 6000 4417 50  0000 C CNN
-F 1 "MCP602" H 6000 4326 50  0000 C CNN
+F 0 "U1" H 6150 4400 50  0000 C CNN
+F 1 "MCP602" H 6150 4300 50  0000 C CNN
 F 2 "" H 6000 4050 50  0001 C CNN
 F 3 "http://ww1.microchip.com/downloads/en/DeviceDoc/21314g.pdf" H 6000 4050 50  0001 C CNN
@@
 U 1 1 5DCF72A8
 P 6000 5000
-F 0 "U1" H 6000 5367 50  0000 C CNN
-F 1 "MCP602" H 6000 5276 50  0000 C CNN
+F 0 "U1" H 6150 5300 50  0000 C CNN
+F 1 "MCP602" H 6150 5200 50  0000 C CNN
 F 2 "" H 6000 5000 50  0001 C CNN
 F 3 "http://ww1.microchip.com/downloads/en/DeviceDoc/21314g.pdf" H 6000 5000 50  0001 C CNN
@@
 L Device:R R6
 U 1 1 5DD42EFB
-P 6000 4350
-F 0 "R6" V 5793 4350 50  0000 C CNN
-F 1 "100k" V 5884 4350 50  0000 C CNN
-F 2 "" V 5930 4350 50  0001 C CNN
-F 3 "~" H 6000 4350 50  0001 C CNN
-	1    6000 4350
+P 6000 4450
+F 0 "R6" V 5793 4450 50  0000 C CNN
+F 1 "100k" V 5884 4450 50  0000 C CNN
+F 2 "" V 5930 4450 50  0001 C CNN
+F 3 "~" H 6000 4450 50  0001 C CNN
+	1    6000 4450
 	0    1    1    0
 $EndComp
 Wire Wire Line
 	5700 4150 5700 4250
-Wire Wire Line
-	5700 4350 5850 4350
-Wire Wire Line
-	6150 4350 6300 4350
-Wire Wire Line
-	6300 4350 6300 4050
 $Comp
 L Device:R R3
@@
 	5300 4250 5700 4250
 Connection ~ 5700 4250
-Wire Wire Line
-	5700 4250 5700 4350
+Connection ~ 6600 2600
+Wire Wire Line
+	6600 2600 7750 2600
+Wire Wire Line
+	6050 2100 6600 2100
+Wire Wire Line
+	6050 2600 6600 2600
+Wire Wire Line
+	6600 2200 6600 2100
+Connection ~ 6600 2100
+Connection ~ 6900 2100
+Wire Wire Line
+	6900 2100 7200 2100
+Wire Wire Line
+	6600 2100 6900 2100
+$Comp
+L LED:IR204A D2
+U 1 1 5DCFF8D1
+P 7800 5750
+F 0 "D2" H 7750 6040 50  0000 C CNN
+F 1 "IR LED" H 7750 5949 50  0000 C CNN
+F 2 "LED_THT:LED_D3.0mm_IRBlack" H 7800 5925 50  0001 C CNN
+F 3 "http://www.everlight.com/file/ProductFile/IR204-A.pdf" H 7750 5750 50  0001 C CNN
+	1    7800 5750
+	0    -1   -1   0
+$EndComp
+Wire Wire Line
+	6300 4450 6150 4450
+Wire Wire Line
+	6300 4050 6300 4450
+Wire Wire Line
+	5700 4450 5850 4450
+Wire Wire Line
+	5700 4250 5700 4450
 $EndSCHEMATC
